File: projects/01-uv-bench/hardware/uv-bench/uv-bench.kicad_pcb (KiCad board)
At the start: 2 copper layers, 58 x 32 mm, 25 parts, among them J1 I2C + 5V (JST-PH), J2 LED star, J3 STDC14 (SWD + VCP), Q1 AO3400A, SW1 PEC09 + push, U1 MCP1700-3.3, U2 STM32C031F6P6

Commit message: UV bench Rev C + remote photodiode head, as ordered at JLCPCB
- Main board Rev C: J4 (JST PH 2-pin) remote photodiode input with
  R6/R8/C8/R7 to PA12 (ADC1_IN12); USART2 on the STDC14 VCP pins;
  rounded corners R 3.5 mm.
- New pd-head project: 12 x 21 mm, SFH 2401 + solder-wire pads with
  strain relief, R 1.5 mm corners.
- Generators parameterised by UVB_DESIGN (design_head/layout_head/
  placement_head build the head).
- interface-spec v2.3 (FB_EXT, MEAS_EXT_PD_RAW, CAL_GAIN_EXT), docs,
  parts list and DigiKey BOM updated for Rev C.
- hardware/fab/2026-10-15-jlcpcb/: the exact Gerber zips uploaded
  (output/ is git-ignored and the autorouter is non-deterministic).

Co-Authored-By: Claude Opus 5.5 <noreply@anthropic.com>
Parts:
- added C8: 100n, Capacitor_SMD:C_0805_2012Metric_Pad1.18x1.45mm_HandSolder, F.Cu at (115.8, 102.5)
- added J4: remote PD (JST-PH), Connector_JST:JST_PH_B2B-PH-K_1x02_P2.00mm_Vertical, F.Cu at (121.2, 102.5)
- added R6: 1k, Resistor_SMD:R_0805_2012Metric_Pad1.20x1.40mm_HandSolder, F.Cu at (124.5, 124.8)
- added R7: 1k, Resistor_SMD:R_0805_2012Metric_Pad1.20x1.40mm_HandSolder, F.Cu at (144.5, 123.8)
- added R8: 10k, Resistor_SMD:R_0805_2012Metric_Pad1.20x1.40mm_HandSolder, F.Cu at (110.8, 102.8)
- moved R4 15.0 mm to (127.0, 122.0), turned to 0 degrees
- moved C7 8.04 mm to (135.0, 125.2)
Connections:
- U2 pad 17: unconnected-(U2-PA10/PA12-Pad17) -> /ADC_EXT_PD
Routing:
- net /EXT_PD: track 0.00 -> 66.2 mm, vias 0 -> 2
- net GND: track 123.8 -> 159.6 mm, vias 13 -> 11
- net /EXT_PD_K: track 0.00 -> 24.5 mm
- net +3V3: track 73.3 -> 57.2 mm, vias 0 -> 2
- net /ADC_EXT_PD: track 0.00 -> 13.4 mm, vias 0 -> 2
- net /SWDIO: track 16.0 -> 22.5 mm
- net /GATE: track 25.7 -> 19.3 mm, vias 2 -> 0
- net /UART_TX: track 13.2 -> 18.4 mm, vias 0 -> 2
- net /UART_RX: track 12.4 -> 17.4 mm, vias 2 -> 4
- net /SDA: track 20.3 -> 15.3 mm
- net /PD: track 28.3 -> 32.0 mm
- net +5V: track 56.3 -> 53.1 mm
- net /I_MON: track 21.7 -> 22.9 mm, vias 0 -> 2
- net /SWCLK: track 14.3 -> 14.9 mm
- net /PWM: track 9.71 -> 10.2 mm
Other:
- board text added: "UV BENCH rev C"
- board text removed: "UV BENCH rev B"
