File: projects/01-uv-bench/hardware/uv-bench/uv-bench.kicad_sch (KiCad schematic)
At the start: 21 parts, among them J1 I2C + 5V (JST-PH), J2 LED star, J3 STDC14 (SWD + VCP), Q1 AO3400A, SW1 PEC09 + push, U1 MCP1700-3.3, U2 STM32C031F6P6

Commit message: UV bench Rev C + remote photodiode head, as ordered at JLCPCB
- Main board Rev C: J4 (JST PH 2-pin) remote photodiode input with
  R6/R8/C8/R7 to PA12 (ADC1_IN12); USART2 on the STDC14 VCP pins;
  rounded corners R 3.5 mm.
- New pd-head project: 12 x 21 mm, SFH 2401 + solder-wire pads with
  strain relief, R 1.5 mm corners.
- Generators parameterised by UVB_DESIGN (design_head/layout_head/
  placement_head build the head).
- interface-spec v2.3 (FB_EXT, MEAS_EXT_PD_RAW, CAL_GAIN_EXT), docs,
  parts list and DigiKey BOM updated for Rev C.
- hardware/fab/2026-10-15-jlcpcb/: the exact Gerber zips uploaded
  (output/ is git-ignored and the autorouter is non-deterministic).

Co-Authored-By: Claude Opus 5.5 <noreply@anthropic.com>
Parts:
- added C8: 100n, Capacitor_SMD:C_0805_2012Metric_Pad1.18x1.45mm_HandSolder, symbol Device:C
- added J4: remote PD (JST-PH), Connector_JST:JST_PH_B2B-PH-K_1x02_P2.00mm_Vertical, symbol Connector_Generic:Conn_01x02
- added R6, R7: 1k, Resistor_SMD:R_0805_2012Metric_Pad1.20x1.40mm_HandSolder, symbol Device:R
- added R8: 10k, Resistor_SMD:R_0805_2012Metric_Pad1.20x1.40mm_HandSolder, symbol Device:R
Connections:
- net +3V3: now also R6.2
- net GND: now also C8.2, R8.2
- net ADC_EXT_PD: now reaches U2.17 (PA10/PA12)
- net ADC_EXT_PD: now also R7.2
- new net EXT_PD: C8.1, J4.2 (Pin_2), R7.1, R8.1
- new net EXT_PD_K: J4.1 (Pin_1), R6.1
- no-connect marks 9 -> 8
Other:
- note added: "8 REMOTE PHOTODIODE (optional, 50 cm cable)"
- title: UV bench Rev B -> UV bench Rev C
